Commit message: Remplacement URDF par la version finale PhantomX

File: hexa_simulation/urdf/hexapode.urdf (robot description, URDF)
Before this commit: robot hexapode_v2, 19 links, 18 joints
Links:
- link base_link: geometry visual box size=0.090 0.055 0.006; visual box size=0.230 0.105 0.010
- link leg_1_coxa_link: geometry visual box size=0.032 0.040 0.030; visual box size=0.052 0.018 0.018
- link leg_1_femur_link: geometry visual box size=0.032 0.040 0.035; visual box size=0.065 0.020 0.016
- link leg_1_tibia_link: geometry visual box size=0.032 0.038 0.032; visual box size=0.045 0.030 0.010
- link leg_2_coxa_link: geometry visual box size=0.032 0.040 0.030; visual box size=0.052 0.018 0.018
- link leg_2_femur_link: geometry visual box size=0.032 0.040 0.035; visual box size=0.065 0.020 0.016
- link leg_2_tibia_link: geometry visual box size=0.032 0.038 0.032; visual box size=0.045 0.030 0.010
- link leg_3_coxa_link: geometry visual box size=0.032 0.040 0.030; visual box size=0.052 0.018 0.018
- link leg_3_femur_link: geometry visual box size=0.032 0.040 0.035; visual box size=0.065 0.020 0.016
- link leg_3_tibia_link: geometry visual box size=0.032 0.038 0.032; visual box size=0.045 0.030 0.010
- link leg_4_coxa_link: geometry visual box size=0.032 0.040 0.030; visual box size=0.052 0.018 0.018
- link leg_4_femur_link: geometry visual box size=0.032 0.040 0.035; visual box size=0.065 0.020 0.016
- link leg_4_tibia_link: geometry visual box size=0.032 0.038 0.032; visual box size=0.045 0.030 0.010
- link leg_5_coxa_link: geometry visual box size=0.032 0.040 0.030; visual box size=0.052 0.018 0.018
- link leg_5_femur_link: geometry visual box size=0.032 0.040 0.035; visual box size=0.065 0.020 0.016
- link leg_5_tibia_link: geometry visual box size=0.032 0.038 0.032; visual box size=0.045 0.030 0.010
- link leg_6_coxa_link: geometry visual box size=0.032 0.040 0.030; visual box size=0.052 0.018 0.018
- link leg_6_femur_link: geometry visual box size=0.032 0.040 0.035; visual box size=0.065 0.020 0.016
- link leg_6_tibia_link: geometry visual box size=0.032 0.038 0.032; visual box size=0.045 0.030 0.010
Joints:
- joint leg_1_coxa_joint: origin xyz=0.13 0.09 0 rpy=0 0 0.65 -> xyz=0.108 0.063 0.000 rpy=0 0 0.524
- joint leg_1_femur_joint: origin xyz=0.09 0 0 rpy=0 0 0 -> xyz=0.052 0 0.000 rpy=0 0 0
- joint leg_1_tibia_joint: origin xyz=0.15 0 -0.05 rpy=0 0 0 -> xyz=0.065 0 -0.035 rpy=0 0 0
- joint leg_2_coxa_joint: origin xyz=0 0.10 0 rpy=0 0 1.57 -> xyz=0.000 0.125 0.000 rpy=0 0 1.570
- joint leg_2_femur_joint: origin xyz=0.09 0 0 -> xyz=0.052 0 0.000 rpy=0 0 0
- joint leg_2_tibia_joint: origin xyz=0.15 0 -0.05 -> xyz=0.065 0 -0.035 rpy=0 0 0
- joint leg_3_coxa_joint: origin xyz=-0.13 0.09 0 rpy=0 0 2.50 -> xyz=-0.108 0.063 0.000 rpy=0 0 2.618
- joint leg_3_femur_joint: origin xyz=0.09 0 0 -> xyz=0.052 0 0.000 rpy=0 0 0
- joint leg_3_tibia_joint: origin xyz=0.15 0 -0.05 -> xyz=0.065 0 -0.035 rpy=0 0 0
- joint leg_4_coxa_joint: origin xyz=0.13 -0.09 0 rpy=0 0 -0.65 -> xyz=0.108 -0.063 0.000 rpy=0 0 -0.524
- joint leg_4_femur_joint: origin xyz=0.09 0 0 -> xyz=0.052 0 0.000 rpy=0 0 0
- joint leg_4_tibia_joint: origin xyz=0.15 0 -0.05 -> xyz=0.065 0 -0.035 rpy=0 0 0
- joint leg_5_coxa_joint: origin xyz=0 -0.10 0 rpy=0 0 -1.57 -> xyz=0.000 -0.125 0.000 rpy=0 0 -1.570
- joint leg_5_femur_joint: origin xyz=0.09 0 0 -> xyz=0.052 0 0.000 rpy=0 0 0
- joint leg_5_tibia_joint: origin xyz=0.15 0 -0.05 -> xyz=0.065 0 -0.035 rpy=0 0 0
- joint leg_6_coxa_joint: origin xyz=-0.13 -0.09 0 rpy=0 0 -2.50 -> xyz=-0.108 -0.063 0.000 rpy=0 0 -2.618
- joint leg_6_femur_joint: origin xyz=0.09 0 0 -> xyz=0.052 0 0.000 rpy=0 0 0
- joint leg_6_tibia_joint: origin xyz=0.15 0 -0.05 -> xyz=0.065 0 -0.035 rpy=0 0 0

Commit message: Update functionnalities

File: hexa_simulation/urdf/hexapode.urdf (robot description, URDF)
Before this commit: robot hexapode_v2, 19 links, 18 joints
Links:
- link base_link: geometry visual box size=0.090 0.055 0.006; visual box size=0.230 0.105 0.010
- link leg_1_coxa_link: geometry visual box size=0.032 0.040 0.030; visual box size=0.052 0.018 0.018
- link leg_1_femur_link: geometry visual box size=0.032 0.040 0.035; visual box size=0.065 0.020 0.016
- link leg_1_tibia_link: geometry visual box size=0.032 0.038 0.032; visual box size=0.045 0.030 0.010
- link leg_2_coxa_link: geometry visual box size=0.032 0.040 0.030; visual box size=0.052 0.018 0.018
- link leg_2_femur_link: geometry visual box size=0.032 0.040 0.035; visual box size=0.065 0.020 0.016
- link leg_2_tibia_link: geometry visual box size=0.032 0.038 0.032; visual box size=0.045 0.030 0.010
- link leg_3_coxa_link: geometry visual box size=0.032 0.040 0.030; visual box size=0.052 0.018 0.018
- link leg_3_femur_link: geometry visual box size=0.032 0.040 0.035; visual box size=0.065 0.020 0.016
- link leg_3_tibia_link: geometry visual box size=0.032 0.038 0.032; visual box size=0.045 0.030 0.010
- link leg_4_coxa_link: geometry visual box size=0.032 0.040 0.030; visual box size=0.052 0.018 0.018
- link leg_4_femur_link: geometry visual box size=0.032 0.040 0.035; visual box size=0.065 0.020 0.016
- link leg_4_tibia_link: geometry visual box size=0.032 0.038 0.032; visual box size=0.045 0.030 0.010
- link leg_5_coxa_link: geometry visual box size=0.032 0.040 0.030; visual box size=0.052 0.018 0.018
- link leg_5_femur_link: geometry visual box size=0.032 0.040 0.035; visual box size=0.065 0.020 0.016
- link leg_5_tibia_link: geometry visual box size=0.032 0.038 0.032; visual box size=0.045 0.030 0.010
- link leg_6_coxa_link: geometry visual box size=0.032 0.040 0.030; visual box size=0.052 0.018 0.018
- link leg_6_femur_link: geometry visual box size=0.032 0.040 0.035; visual box size=0.065 0.020 0.016
- link leg_6_tibia_link: geometry visual box size=0.032 0.038 0.032; visual box size=0.045 0.030 0.010
Joints:
- joint leg_1_coxa_joint: origin xyz=0.13 0.09 0 rpy=0 0 0.65 -> xyz=0.108 0.063 0.000 rpy=0 0 0.524
- joint leg_1_femur_joint: axis 0 1 0 -> 0 -1 0; origin xyz=0.09 0 0 rpy=0 0 0 -> xyz=0.052 0 0.000 rpy=0 0 0
- joint leg_1_tibia_joint: axis 0 1 0 -> 0 -1 0; origin xyz=0.15 0 -0.05 rpy=0 0 0 -> xyz=0.065 0 -0.035 rpy=0 0 0
- joint leg_2_coxa_joint: origin xyz=0 0.10 0 rpy=0 0 1.57 -> xyz=0.000 0.125 0.000 rpy=0 0 1.570
- joint leg_2_femur_joint: axis 0 1 0 -> 0 -1 0; origin xyz=0.09 0 0 -> xyz=0.052 0 0.000 rpy=0 0 0
- joint leg_2_tibia_joint: axis 0 1 0 -> 0 -1 0; origin xyz=0.15 0 -0.05 -> xyz=0.065 0 -0.035 rpy=0 0 0
- joint leg_3_coxa_joint: origin xyz=-0.13 0.09 0 rpy=0 0 2.50 -> xyz=-0.108 0.063 0.000 rpy=0 0 2.618
- joint leg_3_femur_joint: axis 0 1 0 -> 0 -1 0; origin xyz=0.09 0 0 -> xyz=0.052 0 0.000 rpy=0 0 0
- joint leg_3_tibia_joint: axis 0 1 0 -> 0 -1 0; origin xyz=0.15 0 -0.05 -> xyz=0.065 0 -0.035 rpy=0 0 0
- joint leg_4_coxa_joint: origin xyz=0.13 -0.09 0 rpy=0 0 -0.65 -> xyz=0.108 -0.063 0.000 rpy=0 0 -0.524
- joint leg_4_femur_joint: axis 0 1 0 -> 0 -1 0; origin xyz=0.09 0 0 -> xyz=0.052 0 0.000 rpy=0 0 0
- joint leg_4_tibia_joint: axis 0 1 0 -> 0 -1 0; origin xyz=0.15 0 -0.05 -> xyz=0.065 0 -0.035 rpy=0 0 0
- joint leg_5_coxa_joint: origin xyz=0 -0.10 0 rpy=0 0 -1.57 -> xyz=0.000 -0.125 0.000 rpy=0 0 -1.570
- joint leg_5_femur_joint: axis 0 1 0 -> 0 -1 0; origin xyz=0.09 0 0 -> xyz=0.052 0 0.000 rpy=0 0 0
- joint leg_5_tibia_joint: axis 0 1 0 -> 0 -1 0; origin xyz=0.15 0 -0.05 -> xyz=0.065 0 -0.035 rpy=0 0 0
- joint leg_6_coxa_joint: origin xyz=-0.13 -0.09 0 rpy=0 0 -2.50 -> xyz=-0.108 -0.063 0.000 rpy=0 0 -2.618
- joint leg_6_femur_joint: axis 0 1 0 -> 0 -1 0; origin xyz=0.09 0 0 -> xyz=0.052 0 0.000 rpy=0 0 0
- joint leg_6_tibia_joint: axis 0 1 0 -> 0 -1 0; origin xyz=0.15 0 -0.05 -> xyz=0.065 0 -0.035 rpy=0 0 0
